File: esp32-ledmatrix-shield/esp32-ledmatrix-shield.sch (KiCad schematic (older format))
At the start: 22 parts, among them J1 Power, J10 C, J11 D, J12 E, J13 I2C, J14 I2C, J15 Power, J2 JIN, J3 Byp D1, J4 JOUT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

Commit message: schematic and pcb v0.3 devkit support
Parts:
- removed D1: D_Schottky, Diode_THT:D_DO-15_P10.16mm_Horizontal, symbol Device:D_Schottky
- removed J6: CON1 I2C2, Connector_PinHeader_2.54mm:PinHeader_1x06_P2.54mm_Vertical, symbol Connector:Conn_01x06_Male
- removed J7: CON 2, Connector_PinHeader_2.54mm:PinHeader_1x05_P2.54mm_Vertical, symbol Connector:Conn_01x05_Male
- added J10: Ctrl1, Connector_PinHeader_2.54mm:PinHeader_1x04_P2.54mm_Vertical, symbol Connector:Conn_01x04_Male
- added J16: VIN ext, Connector_PinHeader_2.54mm:PinHeader_1x02_P2.54mm_Vertical, symbol Connector:Conn_01x02_Male
- added J5: Ctrl2, Connector_PinHeader_2.54mm:PinHeader_1x04_P2.54mm_Vertical, symbol Connector:Conn_01x04_Male
- added JP1, JP2, JP3, JP4: Jumper, Jumper:SolderJumper-2_P1.3mm_Open_Pad1.0x1.5mm, symbol Device:Jumper
- J11: renamed from J12; footprint Connector_PinHeader_2.54mm:PinHeader_1x03_P2.54mm_Vertical -> Jumper:SolderJumper-3_P1.3mm_Open_Pad1.0x1.5mm
- J6: renamed from J3; value Byp D1 -> VIN ext
- J8: renamed from J10; footprint Connector_PinHeader_2.54mm:PinHeader_1x03_P2.54mm_Vertical -> Jumper:SolderJumper-3_P1.3mm_Open_Pad1.0x1.5mm
- J9: renamed from J11; footprint Connector_PinHeader_2.54mm:PinHeader_1x03_P2.54mm_Vertical -> Jumper:SolderJumper-3_P1.3mm_Open_Pad1.0x1.5mm
- renumbered J9 to J12, J4 to J15, J5 to J2, J2 to J3, J8 to J4, J15 to J7
Connections:
- net labels added: +5V, C', SCL, SCL2, SDA, SDA2
- wire segments 154 -> 152
- no-connect marks 24 -> 28
Other:
- moved on the sheet: J6, J7, R1, R2
