File: ShiftIn-Board/ShiftIn-Board.sch (KiCad schematic (older format))
At the start: 5 parts, among them J1 Conn_01x06_Male, J2 Conn_01x06_Male, J3 Conn_01x08_Male, U1 74HC165_DIL16

Commit message: Shiftin-Board v0.2
Parts:
- U1: footprint Package_SO:SOIC-16_4.55x10.3mm_P1.27mm -> Package_SO:SOIC-16_3.9x9.9mm_P1.27mm
Changed lines of the file:
@@
 F 0 "U1" H 5900 4165 50  0000 C CNN
 F 1 "74HC165_DIL16" H 5900 4074 50  0000 C CNN
-F 2 "Package_SO:SOIC-16_4.55x10.3mm_P1.27mm" H 5900 3450 50  0001 C CNN
+F 2 "Package_SO:SOIC-16_3.9x9.9mm_P1.27mm" H 5900 3450 50  0001 C CNN
 F 3 "DOCUMENTATION" H 5900 3450 50  0001 C CNN
 	1    5900 3450
